File: Hardware/LVDS_to_Dual_EVF/LVDS_to_Dual_EVF.kicad_pcb (KiCad board)
At the start: 2 copper layers, 63 parts, among them J1 Conn_02x15_Odd_Even, J2 FR02C061JA1-R5000, J3 FR02C061JA1-R5000

Commit message: started reverse engineering the EVF pinout
Parts:
- turned J3 to 180 degrees

Commit message: updated schematic
Parts:
- renumbered J2 to J1, J1 to J2, R32 to R10, R43 to R11, R6 to R12, R44 to R13, R7 to R14, R8 to R15, R33 to R16, R45 to R17, R9 to R18, R46 to R19, R1 to R2, R10 to R20, R11 to R21, R34 to R22, R47 to R23, R12 to R24, R48 to R25, R13 to R26, R14 to R27, R35 to R28, R49 to R29, R2 to R3, R15 to R30, R50 to R31, R16 to R32, R17 to R33, R36 to R34, R51 to R35, R18 to R36, R52 to R37, R19 to R38, R20 to R39, R31 to R4, R37 to R40, R53 to R41, R21 to R42, R54 to R43, R22 to R44, R23 to R45, R38 to R46, R55 to R47, R24 to R48, R56 to R49, R41 to R5, R25 to R50, R26 to R51, R39 to R52, R57 to R53, R27 to R54, R58 to R55, R28 to R56, R29 to R57, R40 to R58, R3 to R6, R30 to R60, R60 to R61, R42 to R7, R4 to R8, R5 to R9
Connections:
- J3 pad 1: unconnected-(J3-Pad1) -> GND
- J3 pad 10: unconnected-(J3-Pad10) -> GND
- J3 pad 11: unconnected-(J3-Pad11) -> /VDD9
- J3 pad 12: unconnected-(J3-Pad12) -> /GND0
- J3 pad 14: unconnected-(J3-Pad14) -> /LV2DN
- J3 pad 15: unconnected-(J3-Pad15) -> /LV2DP
- J3 pad 16: unconnected-(J3-Pad16) -> /LV2EN
- J3 pad 17: unconnected-(J3-Pad17) -> /LV2EP
- J3 pad 18: unconnected-(J3-Pad18) -> /LV2CN
- J3 pad 19: unconnected-(J3-Pad19) -> /LV2CP
- J3 pad 2: unconnected-(J3-Pad2) -> /VDD2
- J3 pad 20: unconnected-(J3-Pad20) -> /LV2BN
- J3 pad 21: unconnected-(J3-Pad21) -> /LV2BP
- J3 pad 22: unconnected-(J3-Pad22) -> /LV2AN
- J3 pad 23: unconnected-(J3-Pad23) -> /LV2AP
- J3 pad 24: unconnected-(J3-Pad24) -> /GND0
- J3 pad 25: unconnected-(J3-Pad25) -> GND
- J3 pad 26: unconnected-(J3-Pad26) -> /LVDS1V8
- J3 pad 27: unconnected-(J3-Pad27) -> GND
- J3 pad 28: unconnected-(J3-Pad28) -> GND
- J3 pad 29: unconnected-(J3-Pad29) -> GND
- J3 pad 3: unconnected-(J3-Pad3) -> /VDD3
- J3 pad 30: unconnected-(J3-Pad30) -> GND
- J3 pad 31: unconnected-(J3-Pad31) -> /LVDS1V8
- J3 pad 32: unconnected-(J3-Pad32) -> GND
- J3 pad 33: unconnected-(J3-Pad33) -> GND
- J3 pad 35: unconnected-(J3-Pad35) -> /LV1AP
- J3 pad 36: unconnected-(J3-Pad36) -> /LV1AN
- J3 pad 37: unconnected-(J3-Pad37) -> /LV1BP
- J3 pad 38: unconnected-(J3-Pad38) -> /LV1BN
- J3 pad 39: unconnected-(J3-Pad39) -> /LV1CP
- J3 pad 4: unconnected-(J3-Pad4) -> /VDD6
- J3 pad 40: unconnected-(J3-Pad40) -> /LV1CN
- J3 pad 41: unconnected-(J3-Pad41) -> /LV1EP
- J3 pad 42: unconnected-(J3-Pad42) -> /LV1EN
- J3 pad 43: unconnected-(J3-Pad43) -> /LV1DP
- J3 pad 44: unconnected-(J3-Pad44) -> /LV1DN
- J3 pad 45: unconnected-(J3-Pad45) -> /LVDS1V8
- J3 pad 46: unconnected-(J3-Pad46) -> GND
- J3 pad 47: unconnected-(J3-Pad47) -> Net-(J3-Pad47)
- J3 pad 48: unconnected-(J3-Pad48) -> /LVDS1V8
- J3 pad 49: unconnected-(J3-Pad49) -> GND
- J3 pad 5: unconnected-(J3-Pad5) -> /VDD4
- J3 pad 55: unconnected-(J3-Pad55) -> GND
- J3 pad 56: unconnected-(J3-Pad56) -> GND
- J3 pad 57: unconnected-(J3-Pad57) -> /VDD9
- J3 pad 58: unconnected-(J3-Pad58) -> GND
- J3 pad 59: unconnected-(J3-Pad59) -> /VDD10
- J3 pad 6: unconnected-(J3-Pad6) -> /VDD7
- J3 pad 60: unconnected-(J3-Pad60) -> /VDD2
- J3 pad 61: unconnected-(J3-Pad61) -> GND
- J3 pad 7: unconnected-(J3-Pad7) -> /VDD5
- J3 pad 8: unconnected-(J3-Pad8) -> /VDD8
- J3 pad 9: unconnected-(J3-Pad9) -> /VDD10
