File: Hardware/LVDS_to_Dual_EVF/LVDS_to_Dual_EVF.kicad_sch (KiCad schematic)
At the start: 63 parts, among them J1 Conn_02x15_Odd_Even, J2 FR02C061JA1-R5000, J3 FR02C061JA1-R5000

Commit message: started reverse engineering the EVF pinout
Parts:
- added C1, C10, C11, C12, C13, C2, C3, C4, C5, C6, C7, C8, C9: C, symbol Component_lib:C
- added R1: 0, symbol Component_lib:R
- added R62: R, symbol Component_lib:R
- renumbered J2 to J1, J1 to J2, R32 to R10, R43 to R11, R6 to R12, R44 to R13, R7 to R14, R8 to R15, R33 to R16, R45 to R17, R9 to R18, R46 to R19, R1 to R2, R10 to R20, R11 to R21, R34 to R22, R47 to R23, R12 to R24, R48 to R25, R13 to R26, R14 to R27, R35 to R28, R49 to R29, R2 to R3, R15 to R30, R50 to R31, R16 to R32, R17 to R33, R36 to R34, R51 to R35, R18 to R36, R52 to R37, R19 to R38, R20 to R39, R31 to R4, R37 to R40, R53 to R41, R21 to R42, R54 to R43, R22 to R44, R23 to R45, R38 to R46, R55 to R47, R24 to R48, R56 to R49, R41 to R5, R25 to R50, R26 to R51, R39 to R52, R57 to R53, R27 to R54, R58 to R55, R28 to R56, R29 to R57, R40 to R58, R3 to R6, R30 to R60, R60 to R61, R42 to R7, R4 to R8, R5 to R9
Connections:
- net GND: now reaches J3.1
- net GND: now also J3.10, J3.25, J3.27, J3.28, J3.29, J3.30, J3.32, J3.33, J3.46, J3.49, J3.55, J3.56, J3.58, J3.61, C1.2, C10.2, C11.2, C12.2, C13.2, C2.2, C3.2, C4.2, C5.2, C6.2, C7.2, C8.2, C9.2, R1.2
- net VDD9: now reaches J3.11
- net VDD9: now also J3.57
- net GND0: now reaches J3.12
- net GND0: now also J3.24, R1.1
- net LV2DN: now reaches J3.14
- net LV2DP: now reaches J3.15
- net LV2EN: now reaches J3.16
- net LV2EP: now reaches J3.17
- net LV2CN: now reaches J3.18
- net LV2CP: now reaches J3.19
- net VDD2: now reaches J3.2
- net VDD2: now also J3.60, C2.1, C3.1
- net LV2BN: now reaches J3.20
- net LV2BP: now reaches J3.21
- net LV2AN: now reaches J3.22
- net LV2AP: now reaches J3.23
- net LVDS1V8: now reaches J3.26
- net LVDS1V8: now also J3.31, J3.45, J3.48, C1.1, C10.1
- net VDD3: now reaches J3.3
- net VDD3: now also C4.1
- net LV1AP: now reaches J3.35
- net LV1AN: now reaches J3.36
- net LV1BP: now reaches J3.37
- net LV1BN: now reaches J3.38
- net LV1CP: now reaches J3.39
- net VDD6: now reaches J3.4
- net VDD6: now also C7.1
- net LV1CN: now reaches J3.40
- net LV1EP: now reaches J3.41
- net LV1EN: now reaches J3.42
- net LV1DP: now reaches J3.43
- net LV1DN: now reaches J3.44
- net at J3.47: now also R62.2
- net VDD4: now reaches J3.5
- net VDD4: now also C5.1
- net VDD10: now reaches J3.59
- net VDD10: now also J3.9, C11.1, C12.1, C13.1
- net VDD7: now reaches J3.6
- net VDD7: now also C8.1
- net VDD5: now reaches J3.7
- net VDD5: now also C6.1
- net VDD8: now reaches J3.8
- net VDD8: now also C9.1
Other:
- moved on the sheet: J3

Commit message: updated schematic
Connections:
- net VDD10: no longer J3.59, J3.9
- net VDD2: no longer J3.2
- net VDD3: no longer J3.3
- net VDD6: no longer J3.4
- net VDD7: no longer J3.6
- net VDD8: no longer J3.8
- new net VDD10-9V9: J3.59, J3.9
- new net VDD2-9V: J3.2
- new net VDD3-9V9: J3.3
- new net VDD6-8V2: J3.4
- new net VDD7-7V7: J3.6
- new net VDD8-8V4: J3.8
Other:
- moved on the sheet: J3, R1, R62
